Commit message: 仿真你到底有啥毛病

File: reBotArmController_ROS2/src/rebotarm_moveit_config/config/rebotarm_rs_gazebo.urdf.xacro (robot description, xacro)
@@ -14,4 +14,36 @@
     initial_positions_file="$(arg initial_positions_file)"
     hardware_plugin="gz_ros2_control/GazeboSimSystem"/>
+  <link name="wrist_camera_link">
+    <inertial>
+      <mass value="0.03"/>
+      <inertia ixx="0.00001" ixy="0" ixz="0" iyy="0.00001" iyz="0" izz="0.00001"/>
+    </inertial>
+    <visual>
+      <geometry>
+        <box size="0.05 0.04 0.03"/>
+      </geometry>
+      <material name="rs_base_black"/>
+    </visual>
+    <visual>
+      <origin xyz="0.026 0 0" rpy="0 1.5708 0"/>
+      <geometry>
+        <cylinder radius="0.007" length="0.004"/>
+      </geometry>
+      <material name="wrist_camera_lens">
+        <color rgba="0.08 0.2 0.35 1"/>
+      </material>
+    </visual>
+  </link>
+  <joint name="wrist_camera_mount" type="fixed">
+    <origin xyz="0 0 0.045" rpy="0 1.355 0"/>
+    <parent link="gripper_end"/>
+    <child link="wrist_camera_link"/>
+  </joint>
+  <link name="wrist_camera_optical_frame"/>
+  <joint name="wrist_camera_optical_joint" type="fixed">
+    <origin xyz="0 0 0" rpy="-1.5708 0 -1.5708"/>
+    <parent link="wrist_camera_link"/>
+    <child link="wrist_camera_optical_frame"/>
+  </joint>
   <gazebo>
     <plugin
@@ -21,3 +53,25 @@
     </plugin>
   </gazebo>
+  <gazebo reference="wrist_camera_link">
+    <sensor name="wrist_camera" type="camera">
+      <always_on>true</always_on>
+      <update_rate>30</update_rate>
+      <visualize>true</visualize>
+      <topic>/wrist_camera/image_raw</topic>
+      <camera>
+        <horizontal_fov>1.5708</horizontal_fov>
+        <image>
+          <width>640</width>
+          <height>480</height>
+          <format>R8G8B8</format>
+        </image>
+        <clip>
+          <near>0.05</near>
+          <far>2.0</far>
+        </clip>
+        <camera_info_topic>/wrist_camera/camera_info</camera_info_topic>
+        <optical_frame_id>wrist_camera_optical_frame</optical_frame_id>
+      </camera>
+    </sensor>
+  </gazebo>
 </robot>
