Commit message: 还差相机未部署

File: robot-sim/public/robot/ur_umi_real/urdf/ur5_umi_real.urdf (robot description, URDF)
Before this commit: robot ur5_umi_real, 17 links, 16 joints
Links:
- removed link left_finger_link
- removed link right_finger_link
- removed link umi_base_link
- added link fixed_mount_link; visual mesh filename=package://ur_umi_real/meshes/part_1.stl; visual mesh filename=package://ur_umi_real/meshes/part_2.stl
- added link left_jaw_link; visual mesh filename=package://ur_umi_real/meshes/finger_holder_left.stl; visual mesh filename=package://ur_umi_real/meshes/left_finger.stl
- added link right_jaw_link; visual mesh filename=package://ur_umi_real/meshes/finger_holder_right.stl; visual mesh filename=package://ur_umi_real/meshes/right_finger.stl
Joints:
- removed joint left_finger_joint
- removed joint mount_to_umi
- removed joint right_finger_joint
- added joint left_jaw_joint: type prismatic, parent fixed_mount_link, child left_jaw_link, origin xyz=0 0 0 rpy=0 0 0, axis -1 0 0, limit lower=0 upper=0.055 effort=0 velocity=0
- added joint mount_to_fixed_mount: type fixed, parent mount_link, child fixed_mount_link, origin xyz=0 0 0 rpy=0 0 0
- added joint right_jaw_joint: type prismatic, parent fixed_mount_link, child right_jaw_link, origin xyz=0 0 0 rpy=0 0 0, axis 1 0 0, limit lower=0 upper=0.055 effort=0 velocity=0
- joint ur5_to_mount: origin xyz=0 0 0 rpy=-1.5707963267948966 0 0 -> xyz=0 0 0 rpy=-1.5707963267948966 0 3.141592653589793

Commit message: feat(robot): 将 GoPro 视觉固定到 mount_link

File: robot-sim/public/robot/ur_umi_real/urdf/ur5_umi_real.urdf (robot description, URDF)
Before this commit: robot ur5_cad_mount, 17 links, 16 joints
Links:
- link mount_link: geometry collision mesh filename=package://ur_umi_real/meshes/mount.stl; visual mesh filename=package://ur_umi_real/meshes/gopro.stl

Commit message: feat(robot-sim): 为 UR5_CAD 添加 CAD 抓取 TCP

File: robot-sim/public/robot/ur_umi_real/urdf/ur5_umi_real.urdf (robot description, URDF)
Before this commit: robot ur5_cad_mount, 17 links, 16 joints
Links:
- added link umi_tcp_link
Joints:
- added joint tool0_to_umi_tcp_link: type fixed, parent tool0, child umi_tcp_link, origin xyz=0 -0.003600 0.224785782 rpy=0 0 0
